File: DiodeAdapterSmd/Hardware/DiodeAdapterSmd.kicad_pcb (KiCad board)
At the start: 2 copper layers, 14 x 20 mm, 4 parts, among them P1 LED, P2 LED, X1 CONN_01X02, X2 CONN_01X02

Commit message: changes
Parts:
- X1: renamed from X2; value CONN_01X02 -> Wires
- X2: renamed from X1; value CONN_01X02 -> Wires
Connections:
- net /GND_1 renamed /GND
- net /V+_1 renamed /V+
Changed lines of the file:
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@@
       (drillshape 0)
       (scaleselection 1)
-      (outputdirectory "../../Fabrication/DiodeAdapter/Gerber"))
+      (outputdirectory "Fabrication/Gerber"))
   )
   (net 0 "")
-  (net 1 /V+_1)
-  (net 2 /GND_1)
+  (net 1 /V+)
+  (net 2 /GND)
   (net_class Default "This is the default net class."
     (clearance 0.2)
@@
     (uvia_dia 0.3)
     (uvia_drill 0.1)
-    (add_net /GND_1)
-    (add_net /V+_1)
+    (add_net /GND)
+    (add_net /V+)
   )
   (module EsseivaN_Lib:WirePad_02 (layer F.Cu)
     (at 107 67)
-    (fp_text reference X2 (at -4.5 0 90) (layer F.SilkS) hide
+    (fp_text reference X1 (at -4.5 0 90) (layer F.SilkS) hide
       (effects (font (size 1 1) (thickness 0.15)))
     )
-    (fp_text value CONN_01X02 (at 0 -3.5) (layer F.Fab)
+    (fp_text value Wires (at 0 -3.5) (layer F.Fab)
       (effects (font (size 1 1) (thickness 0.15)))
     )
+    (fp_line (start 3.5 -2.5) (end 3.5 2.5) (layer F.SilkS) (width 0.12))
+    (fp_line (start -3.5 -2.5) (end -3.5 2.5) (layer F.SilkS) (width 0.12))
+    (fp_line (start -3.5 2.5) (end -1 2.5) (layer F.SilkS) (width 0.12))
     (fp_line (start -3.5 -2.5) (end -1 -2.5) (layer F.SilkS) (width 0.12))
-    (fp_line (start -3.5 2.5) (end -1 2.5) (layer F.SilkS) (width 0.12))
-    (fp_line (start -3.5 -2.5) (end -3.5 2.5) (layer F.SilkS) (width 0.12))
-    (fp_line (start 3.5 -2.5) (end 3.5 2.5) (layer F.SilkS) (width 0.12))
     (pad 1 connect rect (at -1.905 0) (size 2 4) (layers F.Cu F.Mask)
-      (net 1 /V+_1))
+      (net 1 /V+))
     (pad 2 connect rect (at 1.905 0) (size 2 4) (layers F.Cu F.Mask)
-      (net 2 /GND_1))
+      (net 2 /GND))
   )
   (module EsseivaN_Lib:WirePad_02 (layer B.Cu)
     (at 107 53)
-    (fp_text reference X1 (at -4.5 0 -90) (layer B.SilkS) hide
+    (fp_text reference X2 (at -4.5 0 -90) (layer B.SilkS) hide
       (effects (font (size 1 1) (thickness 0.15)) (justify mirror))
     )
-    (fp_text value CONN_01X02 (at 0 3.5) (layer B.Fab)
+    (fp_text value Wires (at 0 3.5) (layer B.Fab)
       (effects (font (size 1 1) (thickness 0.15)) (justify mirror))
     )
+    (fp_line (start 3.5 2.5) (end 3.5 -2.5) (layer B.SilkS) (width 0.12))
+    (fp_line (start -3.5 2.5) (end -3.5 -2.5) (layer B.SilkS) (width 0.12))
+    (fp_line (start -3.5 -2.5) (end -1 -2.5) (layer B.SilkS) (width 0.12))
     (fp_line (start -3.5 2.5) (end -1 2.5) (layer B.SilkS) (width 0.12))
-    (fp_line (start -3.5 -2.5) (end -1 -2.5) (layer B.SilkS) (width 0.12))
-    (fp_line (start -3.5 2.5) (end -3.5 -2.5) (layer B.SilkS) (width 0.12))
-    (fp_line (start 3.5 2.5) (end 3.5 -2.5) (layer B.SilkS) (width 0.12))
     (pad 1 connect rect (at -1.905 0) (size 2 4) (layers B.Cu B.Mask)
-      (net 1 /V+_1))
+      (net 1 /V+))
     (pad 2 connect rect (at 1.905 0) (size 2 4) (layers B.Cu B.Mask)
-      (net 2 /GND_1))
+      (net 2 /GND))
   )
   (module EsseivaN_Lib:LED_LH351D (layer F.Cu)
@@
       (effects (font (size 1 1) (thickness 0.15)))
     )
+    (fp_line (start 3.556 -3.556) (end -3.556 -3.556) (layer F.CrtYd) (width 0.15))
+    (fp_line (start -3.556 -3.556) (end -3.556 3.556) (layer F.CrtYd) (width 0.15))
+    (fp_line (start -3.556 3.556) (end 3.556 3.556) (layer F.CrtYd) (width 0.15))
+    (fp_line (start 3.556 3.556) (end 3.556 -3.556) (layer F.CrtYd) (width 0.15))
+    (fp_circle (center 0 0) (end 1.825 0) (layer F.Fab) (width 0.1))
+    (fp_line (start -1.75 1.75) (end -1.75 -1.75) (layer F.Fab) (width 0.1))
+    (fp_line (start -1.75 -1.75) (end 1.75 -1.75) (layer F.Fab) (width 0.1))
+    (fp_line (start 1.75 -1.75) (end 1.75 1.75) (layer F.Fab) (width 0.1))
     (fp_line (start 1.75 1.75) (end -1.75 1.75) (layer F.Fab) (width 0.1))
-    (fp_line (start 1.75 -1.75) (end 1.75 1.75) (layer F.Fab) (width 0.1))
-    (fp_line (start -1.75 -1.75) (end 1.75 -1.75) (layer F.Fab) (width 0.1))
-    (fp_line (start -1.75 1.75) (end -1.75 -1.75) (layer F.Fab) (width 0.1))
-    (fp_circle (center 0 0) (end 1.825 0) (layer F.Fab) (width 0.1))
-    (fp_line (start 3.556 3.556) (end 3.556 -3.556) (layer F.CrtYd) (width 0.15))
-    (fp_line (start -3.556 3.556) (end 3.556 3.556) (layer F.CrtYd) (width 0.15))
-    (fp_line (start -3.556 -3.556) (end -3.556 3.556) (layer F.CrtYd) (width 0.15))
-    (fp_line (start 3.556 -3.556) (end -3.556 -3.556) (layer F.CrtYd) (width 0.15))
     (fp_text user - (at 4.445 1.27 90) (layer F.Fab)
       (effects (font (size 1 1) (thickness 0.15)))
@@
     )
     (pad 2 smd rect (at 0 -2.15 90) (size 6 2) (layers F.Cu F.Paste F.Mask)
-      (net 1 /V+_1))
+      (net 1 /V+))
     (pad 1 smd rect (at 0 2.15 90) (size 6 2) (layers F.Cu F.Paste F.Mask)
-      (net 2 /GND_1))
+      (net 2 /GND))
     (pad 1 smd rect (at 0 0 90) (size 6 1.3) (layers F.Cu F.Paste F.Mask)
-      (net 2 /GND_1))
+      (net 2 /GND))
   )
   (module EsseivaN_Lib:LED_LITTLE_STAR (layer B.Cu)
@@
       (effects (font (size 1 1) (thickness 0.15)) (justify mirror))
     )
+    (fp_line (start 3.048 4.572) (end -3.048 4.572) (layer B.CrtYd) (width 0.15))
+    (fp_line (start -3.048 4.572) (end -3.048 -4.572) (layer B.CrtYd) (width 0.15))
+    (fp_line (start -3.048 -4.572) (end 3.048 -4.572) (layer B.CrtYd) (width 0.15))
+    (fp_line (start 3.048 -4.572) (end 3.048 4.572) (layer B.CrtYd) (width 0.15))
+    (fp_line (start -3 3) (end 3 3) (layer B.Fab) (width 0.15))
+    (fp_line (start 3 3) (end 3 -3) (layer B.Fab) (width 0.15))
+    (fp_line (start 3 -3) (end -3 -3) (layer B.Fab) (width 0.15))
     (fp_line (start -3 -3) (end -3 3) (layer B.Fab) (width 0.15))
-    (fp_line (start 3 -3) (end -3 -3) (layer B.Fab) (width 0.15))
-    (fp_line (start 3 3) (end 3 -3) (layer B.Fab) (width 0.15))
-    (fp_line (start -3 3) (end 3 3) (layer B.Fab) (width 0.15))
-    (fp_line (start 3.048 -4.572) (end 3.048 4.572) (layer B.CrtYd) (width 0.15))
-    (fp_line (start -3.048 -4.572) (end 3.048 -4.572) (layer B.CrtYd) (width 0.15))
-    (fp_line (start -3.048 4.572) (end -3.048 -4.572) (layer B.CrtYd) (width 0.15))
-    (fp_line (start 3.048 4.572) (end -3.048 4.572) (layer B.CrtYd) (width 0.15))
     (fp_text user - (at 4.064 3 90) (layer B.Fab) hide
       (effects (font (size 1 1) (thickness 0.15)) (justify mirror))
@@
     )
     (pad 1 smd rect (at 0 3 90) (size 5.2 3) (layers B.Cu B.Paste B.Mask)
-      (net 2 /GND_1))
+      (net 2 /GND))
     (pad 2 smd rect (at 0 -2.5 90) (size 5.2 4) (layers B.Cu B.Paste B.Mask)
-      (net 1 /V+_1))
+      (net 1 /V+))
   )
   (gr_text "Esseiva Nicolas\nDiode adapter\n24092020 R00" (at 107 66) (layer B.SilkS)
@@
   (segment (start 109.15 60) (end 109.15 53.85) (width 1) (layer F.Cu) (net 2) (status 10))
   (segment (start 110 53) (end 112 53) (width 1) (layer F.Cu) (net 2))
-  (zone (net 2) (net_name /GND_1) (layer F.Cu) (hatch edge 0.508)
+  (zone (net 2) (net_name /GND) (layer F.Cu) (hatch edge 0.508)
     (connect_pads (clearance 0.508))
     (min_thickness 0.254)
@@
     )
   )
-  (zone (net 2) (net_name /GND_1) (layer B.Cu) (hatch edge 0.508)
+  (zone (net 2) (net_name /GND) (layer B.Cu) (hatch edge 0.508)
     (connect_pads (clearance 0.508))
     (min_thickness 0.254)
