File: MRF89XAM8A_Breakout/MRF89XAM8A_Breakout.kicad_pcb (KiCad board)
At the start: 2 copper layers, 39 x 28 mm, 9 parts, among them J1 Connector, U1 MRF89XAM8A, X1 CONN_1_to_6, X2 CONN_7_to_12

Commit message: changes
Other:
- board text added: "MRF89XAM8A Breakout EsseivaN - V1 13.10.2020"
Changed lines of the file:
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@@
   (general
     (thickness 1.6)
-    (drawings 4)
+    (drawings 5)
     (tracks 187)
     (zones 0)
@@
     (visible_elements 7FFFFFFF)
     (pcbplotparams
-      (layerselection 0x010fc_ffffffff)
+      (layerselection 0x010f0_ffffffff)
       (usegerberextensions false)
       (usegerberattributes true)
@@
       (outputformat 1)
       (mirror false)
-      (drillshape 1)
+      (drillshape 0)
       (scaleselection 1)
-      (outputdirectory ""))
+      (outputdirectory "Fabrication/Gerber/"))
   )
   (net 0 "")
@@
       (effects (font (size 1 1) (thickness 0.15)) (justify mirror))
     )
-    (fp_text user %R (at 0 1.75 270) (layer B.Fab)
-      (effects (font (size 1 1) (thickness 0.15)) (justify mirror))
-    )
     (fp_line (start -1 -0.62) (end -1 0.62) (layer B.Fab) (width 0.1))
     (fp_line (start 1 -0.62) (end -1 -0.62) (layer B.Fab) (width 0.1))
@@
     (fp_line (start 2.25 -0.87) (end 2.25 0.88) (layer B.CrtYd) (width 0.05))
     (fp_line (start 2.25 -0.87) (end -2.25 -0.87) (layer B.CrtYd) (width 0.05))
+    (fp_text user %R (at 0 1.75 270) (layer B.Fab)
+      (effects (font (size 1 1) (thickness 0.15)) (justify mirror))
+    )
     (pad 1 smd rect (at -1.25 0 90) (size 1.5 1.25) (layers B.Cu B.Paste B.Mask)
       (net 2 VCC_3V3))
@@
     )
     (fp_text value 4.7uF (at 0 1.75 90) (layer F.Fab)
-      (effects (font (size 1 1) (thickness 0.15)))
-    )
-    (fp_text user %R (at 0 -1.75 90) (layer F.Fab)
       (effects (font (size 1 1) (thickness 0.15)))
     )
@@
     (fp_line (start 2.25 0.87) (end 2.25 -0.88) (layer F.CrtYd) (width 0.05))
     (fp_line (start 2.25 0.87) (end -2.25 0.87) (layer F.CrtYd) (width 0.05))
+    (fp_text user %R (at 0 -1.75 90) (layer F.Fab)
+      (effects (font (size 1 1) (thickness 0.15)))
+    )
     (pad 1 smd rect (at -1.25 0 90) (size 1.5 1.25) (layers F.Cu F.Paste F.Mask)
       (net 2 VCC_3V3))
@@
       (effects (font (size 1 1) (thickness 0.15)) (justify mirror))
     )
-    (fp_text user %R (at 0 -6.35 270) (layer B.Fab)
-      (effects (font (size 1 1) (thickness 0.15)) (justify mirror))
-    )
     (fp_line (start -0.635 1.27) (end 1.27 1.27) (layer B.Fab) (width 0.1))
     (fp_line (start 1.27 1.27) (end 1.27 -13.97) (layer B.Fab) (width 0.1))
@@
     (fp_line (start 1.8 -14.5) (end 1.8 1.8) (layer B.CrtYd) (width 0.05))
     (fp_line (start 1.8 1.8) (end -1.8 1.8) (layer B.CrtYd) (width 0.05))
+    (fp_text user %R (at 0 -6.35 270) (layer B.Fab)
+      (effects (font (size 1 1) (thickness 0.15)) (justify mirror))
+    )
     (pad 1 thru_hole rect (at 0 0 180) (size 1.7 1.7) (drill 1) (layers *.Cu *.Mask)
       (net 3 GND))
@@
     )
     (fp_text value CONN_7_to_12 (at 0 -15.03) (layer B.Fab)
-      (effects (font (size 1 1) (thickness 0.15)) (justify mirror))
-    )
-    (fp_text user %R (at 0 -6.35 270) (layer B.Fab)
       (effects (font (size 1 1) (thickness 0.15)) (justify mirror))
     )
@@
     (fp_line (start 1.8 -14.5) (end 1.8 1.8) (layer B.CrtYd) (width 0.05))
     (fp_line (start 1.8 1.8) (end -1.8 1.8) (layer B.CrtYd) (width 0.05))
+    (fp_text user %R (at 0 -6.35 270) (layer B.Fab)
+      (effects (font (size 1 1) (thickness 0.15)) (justify mirror))
+    )
     (pad 1 thru_hole rect (at 0 0 180) (size 1.7 1.7) (drill 1) (layers *.Cu *.Mask)
       (net 9 /SDO))
@@
     )
   )
+  (gr_text "MRF89XAM8A Breakout\nEsseivaN - V1\n13.10.2020" (at 102 90) (layer B.SilkS)
+    (effects (font (size 1.5 1.5) (thickness 0.3)) (justify mirror))
+  )
   (gr_line (start 81.5 83.5) (end 81.5 111.5) (layer Edge.Cuts) (width 0.05))
